Commit message: new doubt

File: catkin_ws/src/my_robot/urdf/my_robot.xacro (robot description, xacro)
@@ -1,58 +1,5 @@
 <?xml version='1.0'?>
 <robot name="my_robot" xmlns:xacro="http://www.ros.org/wiki/xacro">
-<link name="left_wheel">
-    <visual>
-        <origin xyz="0 0 0" rpy="0 1.5707 1.5707" />
-        <geometry>
-            < cylinder radius="0.1" length="0.05"/>
-        </geometry>
-    </visual>
-    <collision>
-        <origin xyz="0 0 0" rpy="0 1.5707 1.5707" />
-        <geometry>
-            < cylinder radius="0.1" length="0.05"/>
-        </geometry>
-    </collision>
-    <inertia>
-        <origin xyz="0 0 0" rpy="0 1.5707 1.5707" />
-        <mass value="5" />
-        <inertia ixx="0.1" ixy="0" ixz="0" iyy="0.1" iyz="0" izz="0.1" />
-    </inertia>
-</link>
-<link name="right_wheel">
-    <visual>
-        <origin xyz="0 0 0" rpy="0 1.5707 1.5707" />
-        <geometry>
-            < cylinder radius="0.1" length="0.05"/>
-        </geometry>
-    </visual>
-    <collision>
-        <origin xyz="0 0 0" rpy="0 1.5707 1.5707" />
-        <geometry>
-            < cylinder radius="0.1" length="0.05"/>
-        </geometry>
-    </collision>
-    <inertia>
-        <origin xyz="0 0 0" rpy="0 1.5707 1.5707" />
-        <mass value="5" />
-        <inertia ixx="0.1" ixy="0" ixz="0" iyy="0.1" iyz="0" izz="0.1" />
-    </inertia>
-</link>
- <joint type="continuous" name="left_wheel_hinge">
-    <origin xyz="0 0.15 0" rpy="0 0 0"/>
-    <child link="left_wheel"/>
-    <parent link="chassis"/>
-    <axis xyz="0 1 0" rpy="0 0 0"/>
-    <limit effort="10000" velocity="1000"/>
-    <dynamics damping="1.0" friction="1.0"/>
-  </joint>
- <joint type="continuous" name="right_wheel_hinge">
-    <origin xyz="0 -0.15 0" rpy="0 0 0"/>
-    <child link="right_wheel"/>
-    <parent link="chassis"/>
-    <axis xyz="0 1 0" rpy="0 0 0"/>
-    <limit effort="10000" velocity="1000"/>
-    <dynamics damping="1.0" friction="1.0"/>
-  </joint>
+	<xacro:include filename="$(find my_robot)/urdf/my_robot.gazebo" />
   <link name="robot_footprint"></link>
   <joint name="robot_footprint_joint" type="fixed">
@@ -109,3 +56,124 @@
     </visual>
   </link>
+<link name="left_wheel">
+    <inertial>
+      <mass value="5.0" />
+      <origin xyz="0 0 0" rpy="0 1.5707 1.5707" />
+      <inertia
+        ixx="0.1" ixy="0" ixz="0"
+        iyy="0.1" iyz="0"
+        izz="0.1"
+      />
+    </inertial>
+    <collision>
+      <origin xyz="0 0 0" rpy="0 1.5707 1.5707" />
+      <geometry>
+        <cylinder radius="0.1" length="0.05" />
+      </geometry>
+    </collision>
+    <visual>
+      <origin xyz="0 0 0" rpy="0 1.5707 1.5707" />
+      <geometry>
+        <cylinder radius="0.1" length="0.05" />
+      </geometry>
+    </visual>
+  </link>
+  <link name="right_wheel">
+    <inertial>
+      <mass value="5.0" />
+      <origin xyz="0 0 0" rpy="0 1.5707 1.5707" />
+      <inertia
+        ixx="0.1" ixy="0" ixz="0"
+        iyy="0.1" iyz="0"
+        izz="0.1"
+      />
+    </inertial>
+    <collision>
+      <origin xyz="0 0 0" rpy="0 1.5707 1.5707" />
+      <geometry>
+        <cylinder radius="0.1" length="0.05" />
+      </geometry>
+    </collision>
+    <visual>
+      <origin xyz="0 0 0" rpy="0 1.5707 1.5707" />
+      <geometry>
+        <cylinder radius="0.1" length="0.05" />
+      </geometry>
+    </visual>
+  </link>
+<joint type="continuous" name="left_wheel_hinge">
+    <origin xyz="0 0.15 0" rpy="0 0 0" />
+    <child link="left_wheel" />
+    <parent link="chassis" />
+    <axis xyz="0 1 0" rpy="0 0 0" />
+    <limit effort="10000" velocity="1000" />
+    <dynamics damping="1.0" friction="1.0" />
+  </joint>
+  <joint type="continuous" name="right_wheel_hinge">
+    <origin xyz="0 -0.15 0" rpy="0 0 0" />
+    <child link="right_wheel" />
+    <parent link="chassis" />
+    <axis xyz="0 1 0" rpy="0 0 0" />
+    <limit effort="10000" velocity="1000" />
+    <dynamics damping="1.0" friction="1.0" />
+  </joint>
+<link name="camera">
+	<inertial>
+      <mass value="0.1" />
+      <origin xyz="0 0 0" rpy="0 0 0" />
+	<box_inertia m="0.1" x="0.05" y="0.05" z="0.05"/>
+      <inertia
+        ixx="1e-6" ixy="0" ixz="0"
+        iyy="1e-6" iyz="0"
+        izz="1e-6"
+      />
+    </inertial>
+    <collision>
+      <origin xyz="0 0 0" rpy="0 0 0" />
+      <geometry>
+        <box  size="0.05 0.05 0.05"/>
+      </geometry>
+    </collision>
+    <visual>
+     <origin xyz="0 0 0" rpy="0 0 0" />
+      <geometry>
+        <box  size="0.05 0.05 0.05"/>
+      </geometry>
+    </visual>
+</link>
+<joint type="fixed" name="camera_joint">
+    <origin xyz="0.2 0 0" rpy="0 0 0" />
+    <child link="camera" />
+    <parent link="chassis" />
+    <axis xyz="0 1 0"/>
+</joint>
+<link name="hokuyo">
+<inertial>
+      <mass value="1e-5" />
+      <origin xyz="0 0 0" rpy="0 0 0" />
+      <inertia
+        ixx="1e-6" ixy="0" ixz="0"
+        iyy="1e-6" iyz="0"
+        izz="1e-6"
+      />
+    </inertial>
+    <collision>
+      <origin xyz="0 0 0" rpy="0 0 0" />
+      <geometry>
+        <box  size="0.1 0.1 0.1"/>
+      </geometry>
+    </collision>
+    <visual>
+     <origin xyz="0 0 0" rpy="0 0 0" />
+      <geometry>
+        <mesh filename="package://my_robot/meshes/hokuyo.dae" />
+      </geometry>
+    </visual>
+</link>
+<joint type="fixed" name="hokuyo_joint">
+    <origin xyz="0.15 0 .1" rpy="0 0 0" />
+    <child link="hokuyo" />
+    <parent link="chassis" />
+    <axis xyz="0 1 0"/>
+</joint>
 </robot>

Commit message: why aren't the wheel color changing

File: catkin_ws/src/my_robot/urdf/my_robot.xacro (robot description, xacro)
@@ -102,4 +102,10 @@
     </visual>
   </link>
+<gazebo reference="left_wheel">
+  <material>Gazebo/Blue</material>
+</gazebo>
+<gazebo reference="right_wheel">
+  <material>Gazebo/Red</material>
+</gazebo>
 <joint type="continuous" name="left_wheel_hinge">
     <origin xyz="0 0.15 0" rpy="0 0 0" />
